File: dev1/openacqu-dev1/openacqu-dev1.kicad_pcb (KiCad board)
At the start: 4 copper layers, 45 x 36 mm, 35 parts, among them J1 GSB1C41110SSHR, J2 Test Points, U1 MCP2221AT-I_ML, U2 LP5817DRLR, U3 FXL6408UMX, U4 24AA025E48T-E_OT, U5 AP2112K-3.3TRG1, U6 TPS22996HQDYCRQ1

Commit message: Placement and routing complete for DEV1
Parts:
- added J3: 77313-118-16LF, openacqu_footprints:AMPHENOL_77313-118-16LF, F.Cu at (102.0, 75.0)
Connections:
- U3 pad 11: unconnected-(U3-GPIO1-Pad11) -> Net-(U3-GPIO1)
- U3 pad 12: unconnected-(U3-GPIO0-Pad12) -> Net-(U3-GPIO0)
- U3 pad 3: unconnected-(U3-GPIO7-Pad3) -> Net-(U3-GPIO7)
- U3 pad 4: unconnected-(U3-GPIO6-Pad4) -> Net-(U3-GPIO6)
- U3 pad 5: unconnected-(U3-GPIO5-Pad5) -> Net-(U3-GPIO5)
- U3 pad 6: unconnected-(U3-GPIO4-Pad6) -> Net-(U3-GPIO4)
- U3 pad 7: unconnected-(U3-GPIO3-Pad7) -> Net-(U3-GPIO3)
- U3 pad 8: unconnected-(U3-GPIO2-Pad8) -> Net-(U3-GPIO2)
Routing:
- net Net-(U3-GPIO2): track 0.00 -> 36.6 mm
- net Net-(U3-GPIO3): track 0.00 -> 35.4 mm
- net Net-(U3-GPIO4): track 0.00 -> 34.1 mm
- net Net-(U3-GPIO5): track 0.00 -> 32.9 mm
- net Net-(U3-GPIO6): track 0.00 -> 32.2 mm
- net Net-(U3-GPIO0): track 0.00 -> 32.2 mm
- net Net-(U3-GPIO7): track 0.00 -> 32.1 mm
- net Net-(U3-GPIO1): track 0.00 -> 30.6 mm
- net GND: vias 27 -> 70
Other:
- board text added: "DEV1-R01"
- board text added: "HW ID BITS 0 1 2 3 4 5 6 7"
